File: i_n_c_u_r_pcb/incur_board.kicad_pcb (KiCad board)
At the start: 2 copper layers, 100 x 100 mm, 38 parts, among them J1 CV_IN_0, J2 CV_IN_1, J3 CV_IN_2, J4 CV_IN_3, J5 MIDI_DIN_IN, J6 Conn_01x01, J7 VIDEO_OUT, J8 Raspberry_Pi_2_3, U1 MCP3208, U2 6N138

Commit message: incur pcb revision
Parts:
- D1, D2, D3, D4, D5, D6, D7, D8: value BAT85 -> BAT46
- J1: value CV_IN_0 -> mono_jack_3.5mm
- J2: value CV_IN_1 -> mono_jack_3.5mm
- J3: value CV_IN_2 -> mono_jack_3.5mm
- J4: value CV_IN_3 -> mono_jack_3.5mm
- J5: value MIDI_DIN_IN -> din5; footprint SD-50BV:CUI_SD-50BV -> lib_fp:tht_vertical_din5
- J7: value VIDEO_OUT -> rca; footprint RCJ-024:CUI_RCJ-024 -> lib_fp:tht_rca_vertical
- J8: value Raspberry_Pi_2_3 -> 2x20_Extra_Tall_Header; footprint Pin_Headers:Pin_Header_Straight_2x20_Pitch2.54mm -> Connector_PinHeader_2.54mm:PinHeader_2x20_P2.54mm_Vertical
- RV1: value POT_IN_0 -> 10k_pot; footprint Potentiometers:Potentiometer_Alps_RK09K_Horizontal -> lib_fp:tht_vertical_potentiometer
- RV2: value POT_IN_1 -> 10k_pot; footprint Potentiometers:Potentiometer_Alps_RK09K_Horizontal -> lib_fp:tht_vertical_potentiometer
- RV3: value POT_IN_2 -> 10k_pot; footprint Potentiometers:Potentiometer_Alps_RK09K_Horizontal -> lib_fp:tht_vertical_potentiometer
- RV4: value POT_IN_3 -> 10k_pot; footprint Potentiometers:Potentiometer_Alps_RK09K_Horizontal -> lib_fp:tht_vertical_potentiometer
- U1: value MCP3208 -> MCP3008
Connections:
- J7 pad 2: Net-(J6-Pad1) -> GND
Other:
- board text added: "_^ 02"
- board text added: "underscores.shop"
